Commit message: tuning nav

File: urdf/outdoor_bot.urdf (robot description, URDF)
Before this commit: robot autoBot, 17 links, 16 joints
Links:
- removed link digcam_front_link
- removed link digcam_rear_link
- removed link hokuyo_rear_link
- added link digcam_link; visual box size=0.02 .07 .06
- added link hokuyo_right_link; visual cylinder length=0.08 radius=0.035
- added link zoom_digcam_link; visual box size=0.02 .07 .06
Joints:
- removed joint digcam_front_joint
- removed joint digcam_rear_joint
- removed joint hokuyo_rear_joint
- added joint digcam_joint: type fixed, parent front_sensor_bar_link, child digcam_link, origin xyz=0. -0.2 0.03 rpy=0 0 0
- added joint hokuyo_right_joint: type fixed, parent front_sensor_bar_link, child hokuyo_right_link, origin xyz=-0.05 -0.55 0.05 rpy=0 0 -0.78
- added joint zoom_digcam_joint: type fixed, parent front_sensor_bar_link, child zoom_digcam_link, origin xyz=0. 0.2 0.03 rpy=0 0 0
- joint hokuyo_front_joint: origin xyz=0.6 0.49 0.05 rpy=0 0 0 -> xyz=-0.05 0.49 0.05 rpy=0 0 0; parent base_link -> front_sensor_bar_link
- joint webcam_front_joint: origin xyz=0. -0.13 0.03 rpy=0 0 0 -> xyz=0. 0.0 0.03 rpy=0 0 0

Commit message: working out servo bugs

File: urdf/outdoor_bot.urdf (robot description, URDF)
Before this commit: robot autoBot, 17 links, 16 joints
Joints:
- joint hokuyo_front_joint: origin xyz=-0.05 0.49 0.05 rpy=0 0 0 -> xyz=-0.05 0.49 0.05 rpy=1.57 0 0

Commit message: setting up states that search for and move to targets

File: urdf/outdoor_bot.urdf (robot description, URDF)
Before this commit: robot autoBot, 17 links, 16 joints
Joints:
- joint hokuyo_front_joint: origin xyz=-0.05 0.49 0.05 rpy=1.57 0 0 -> xyz=0.05 0.0 0.05 rpy=3.14 0 0
